Commit message: Almost a pre-alpha release

File: rob9/urdf/onearm_backup.urdf.xacro (robot description, xacro)
@@ -74,5 +74,5 @@
   <xacro:include filename="$(find dummy)/urdf/robotiq-3f-gripper_articulated.urdf.xacro"/>
   <joint name="s_model_gripper" type="fixed">
-    <origin xyz="0.0 0.0 0.0" rpy="${pi} 0 0"/>
+    <origin xyz="0.0 0.0 0.0" rpy="0 0 0"/>
     <parent link="flange" />
     <child link="s_connector_plate" />
