Commit message: update moveit_config

File: rob9/urdf/onearm.urdf.xacro (robot description, xacro)
@@ -88,3 +88,23 @@
     <origin xyz="0 0 0" rpy="0 0 0" />
   </xacro:sensor_d435>
+  <link name="top_table">
+    <visual>
+      <geometry>
+        <box size="0.4 0.4 0.4345"/>
+      </geometry>
+      <origin rpy="0 0 0" xyz="0 0 0.0"/>
+      <material name="white"/>
+    </visual>
+    <collision>
+      <geometry>
+        <box size="0.4 0.4 0.4345"/>
+      </geometry>
+      <origin rpy="0 0 0" xyz="0 0 0.0"/>
+    </collision>
+  </link>
+  <joint name="top_table_table_joint" type="fixed">
+    <parent link="table"/>
+    <child link="top_table"/>
+    <origin xyz="0 0 0.717" rpy="0 0 0"/>
+  </joint>
 </robot>

Commit message: FIX: gripper controller and trajectory server

File: rob9/urdf/onearm.urdf.xacro (robot description, xacro)
@@ -7,4 +7,7 @@
   <material name="white">
      <color rgba="1 1 1 1"/>
+  </material>
+  <material name="blue">
+     <color rgba="0 0 1 1"/>
   </material>
   <link name="world" />
@@ -94,5 +97,5 @@
       </geometry>
       <origin rpy="0 0 0" xyz="0 0 0.0"/>
-      <material name="white"/>
+      <material name="blue"/>
     </visual>
     <collision>
