Commit message: ADD: various changes

File: rob9/urdf/onearm_backup_v2.urdf.xacro (robot description, xacro)
@@ -91,16 +91,15 @@
     <origin xyz="0 0 0" rpy="0 0 0" />
   </xacro:sensor_d435>
-  <!-- <box size="0.4 0.4 0.4345"/> -->
   <link name="top_table">
     <visual>
       <geometry>
-        <box size="0.4 0.4 0.43"/>
+        <box size="0.4 0.4 0.4345"/>
       </geometry>
       <origin rpy="0 0 0" xyz="0 0 0.0"/>
-      <material name="aluminum"/>
+      <material name="blue"/>
     </visual>
     <collision>
       <geometry>
-        <box size="0.4 0.4 0.43"/>
+        <box size="0.4 0.4 0.4345"/>
       </geometry>
       <origin rpy="0 0 0" xyz="0 0 0.0"/>
@@ -112,25 +111,3 @@
     <origin xyz="0 0 0.717" rpy="0 0 0"/>
   </joint>
----------------------------------------------
----------------------------------------------
---------------------------------------------
-<link name="connector_box_camera">
-  <visual>
-    <geometry>
-      <box size="0.05 0.05 0.05"/>
-    </geometry>
-    <origin rpy="0 0 0" xyz="0 0 0.0"/>
-  </visual>
-  <collision>
-    <geometry>
-      <box size="0.05 0.05 0.05"/>
-    </geometry>
-    <origin rpy="0 0 0" xyz="0 0 0.0"/>
-  </collision>
-</link>
-<joint name="connector_box_camera" type="fixed">
-  <parent link="ptu_camera_right_ir_frame"/>
-  <child link="connector_box_camera"/>
-  <origin xyz="0 0 0" rpy="0 0 0"/>
-</joint>
 </robot>
