Commit message: Updated the gripper's urdf

File: rob9/urdf/robotiq-3f-gripper_articulated.urdf.xacro (robot description, xacro)
@@ -19,4 +19,10 @@
   </link>
   <link name="gripper_connector_box">
+    <visual>
+      <geometry>
+        <box size="0.05 0.05 0.07"/>
+      </geometry>
+      <origin xyz="0.0 0.0 0.0"/>
+    </visual>
     <collision>
       <geometry>
